File: Touch_Keyboard_10x12_Matrix.kicad_sch (KiCad schematic)
At the start: 583 parts, among them J12 Conn_01x04, J2 Conn_01x02, J5 USB_C_Receptacle_USB2.0, M61 MX_SW_solder, SW1 RotaryEncoder_Switch, SW2 RotaryEncoder_Switch, T1 TOOLINGHOLE, T2 TOOLINGHOLE, T3 TOOLINGHOLE, U1 NCP1117-3.3_SOT223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

Commit message: Initial Design for Review
KiCAD files for a custom mechanical keyboard PCB, with 100%+ layout, dual i2c breakouts, dual alternate rotary encoders, and five hardwired touch sensors, as well as ARGB LEDs.
Parts:
- removed RUN1: Conn_01x01_Pin, TestPoint:TestPoint_Pad_1.0x1.0mm, symbol Touch_Keyboard_Symbols:Conn_01x01_Pin
- added JP3: SolderJumper_2_Bridged, Jumper:SolderJumper-2_P1.3mm_Bridged_RoundedPad1.0x1.5mm, symbol Jumper:SolderJumper_2_Bridged
- Y1: footprint RP2040_minimal:Crystal_SMD_HC49-US -> Touch_Keyboard_Footprints:Crystal_SMD_HC49-US
Connections:
- net +3V3: now also JP3.2 (B)
- net at U3.26 (RUN): now also JP3.1 (A)
Other:
- moved on the sheet: 3V3_PAD1, FID1, FID2, FID3, FID4, GND_PAD1, J12, JP1, JP2, R13, R9
